File: protector_40_pins.kicad_pcb (KiCad board)
At the start: 2 copper layers, 25.4 x 66 mm, 2 parts, among them U1 Alinx_J15, U2 Alinx_J15

Commit message: update
Other:
- board text added: "-GND-5V-"
Changed lines of the file:
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@@
     (property "Sheetfile" "protector_40_pins.kicad_sch")
     (property "Sheetname" "")
-    (fp_text reference "U2" (at -26.63 0) (layer "F.SilkS")
+    (fp_text reference "U2" (at -26.982 0) (layer "F.SilkS")
       (effects (font (size 1 1) (thickness 0.15)))
     )
@@
     (property "Sheetfile" "protector_40_pins.kicad_sch")
     (property "Sheetname" "")
-    (fp_text reference "U1" (at -26.63 0) (layer "F.SilkS")
+    (fp_text reference "U1" (at -26.982 0) (layer "F.SilkS")
       (effects (font (size 1 1) (thickness 0.15)))
     )
@@
     (effects (font (size 1.5 1.5) (thickness 0.3)))
   )
-  (gr_text "39" (at 127.3858 123.756) (layer "F.SilkS")
+  (gr_text "39" (at 127.3858 123.952) (layer "F.SilkS")
     (effects (font (size 1 1) (thickness 0.15)))
   )
@@
     (effects (font (size 1 1) (thickness 0.15)))
   )
-  (gr_text "40\n" (at 129.9258 123.756) (layer "F.SilkS")
+  (gr_text "39" (at 142.748 123.952) (layer "F.SilkS")
+    (effects (font (size 1 1) (thickness 0.15)))
+  )
+  (gr_text "40\n" (at 129.9258 123.952) (layer "F.SilkS")
     (effects (font (size 1 1) (thickness 0.15)))
   )
@@
     (effects (font (size 2 2) (thickness 0.15)))
   )
+  (gr_text "-GND-5V-\n\n" (at 136.398 73.406) (layer "F.SilkS")
+    (effects (font (size 1.5 1) (thickness 0.25)))
+  )
+  (gr_text "40\n" (at 145.288 123.952) (layer "F.SilkS")
+    (effects (font (size 1 1) (thickness 0.15)))
+  )
   (gr_text "ext board\n" (at 133.7358 125.788) (layer "F.SilkS")

Commit message: update
Routing:
- net +5V: track 17.3 -> 0.00 mm
- added copper zone on F.Cu, net +5V
